File: kicad/sensor/sensor.kicad_sch (KiCad schematic)
At the start: 6 parts, among them J1 CONN, U1 150, U2 152, U3 153, U4 156, U5 155

Commit message: add sensor sch
Connections:
- net 157 is gone; now on net 155: U5.6 (INH)
Changed lines of the file:
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@@
     (effects (font (size 1.27 1.27)) (justify left bottom))
   )
-  (label "157" (at 233.045 38.735 0)
+  (label "155" (at 233.045 38.735 0)
     (effects (font (size 1.27 1.27)) (justify left bottom))
   )

Commit message: add kicad plugin
Connections:
- net VCC is gone; now on net VDD: J1.7 (Pin_7), J1.8 (Pin_8)
Changed lines of the file:
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@@
     (pin "9")
-  )
-  (symbol (lib_id "power:VCC") (at 38.735 110.49 0) (unit 1)
-    (in_bom yes) (on_board yes) (fields_autoplaced)
-    (property "Reference" "#PWR02" (id 0) (at 38.735 114.3 0)
-      (effects (font (size 1.27 1.27)) hide)
-    )
-    (property "Value" "VCC" (id 1) (at 38.735 104.775 0))
-    (property "Footprint" "" (id 2) (at 38.735 110.49 0)
-      (effects (font (size 1.27 1.27)) hide)
-    )
-    (property "Datasheet" "" (id 3) (at 38.735 110.49 0)
-      (effects (font (size 1.27 1.27)) hide)
-    )
-    (pin "1")
   )
   (symbol (lib_id "Connector:Conn_01x18_Male") (at 54.61 106.68 180) (unit 1)
@@
     (pin "1")
   )
+  (symbol (lib_id "power:VDD") (at 38.735 110.49 0) (unit 1)
+    (in_bom yes) (on_board yes) (fields_autoplaced)
+    (property "Reference" "#PWR?" (id 0) (at 38.735 114.3 0)
+      (effects (font (size 1.27 1.27)) hide)
+    )
+    (property "Value" "VDD" (id 1) (at 38.735 104.775 0))
+    (property "Footprint" "" (id 2) (at 38.735 110.49 0)
+      (effects (font (size 1.27 1.27)) hide)
+    )
+    (property "Datasheet" "" (id 3) (at 38.735 110.49 0)
+      (effects (font (size 1.27 1.27)) hide)
+    )
+    (pin "1")
+  )
   (symbol (lib_id "power:GND") (at 279.4 51.435 0) (unit 1)
     (in_bom yes) (on_board yes) (fields_autoplaced)
@@
       (reference "#PWR01") (unit 1) (value "VSS") (footprint "")
     )
-    (path "/3f38011c-507a-43b1-879a-76755d092a1c"
-      (reference "#PWR02") (unit 1) (value "VCC") (footprint "")
-    )
     (path "/19c3acc7-fe52-4649-a083-48757cabf659"
       (reference "#PWR03") (unit 1) (value "GND") (footprint "")
@@
       (reference "#PWR023") (unit 1) (value "GND") (footprint "")
     )
+    (path "/c543cf62-eba2-4cb9-ad27-421de95a7000"
+      (reference "#PWR?") (unit 1) (value "VDD") (footprint "")
+    )
     (path "/4193d326-7d2c-4e37-b201-823ceef469b0"

Commit message: script update
Parts:
- added U10, U11, U12, U13, U14, U15, U16, U17, U18, U19, U20, U21, U22, U23, U24, U25, U26, U27, U28, U29, U30, U31, U32, U33, U34, U35, U36, U37, U38, U6, U7, U8, U9: jumper, jumper:jumper, symbol jumper:jumper
Connections:
- net GND: now also U10.2, U11.2, U12.2, U13.2, U14.2, U15.2, U16.2, U17.2, U18.2, U19.2, U20.2, U21.2, U22.2, U23.2, U24.2, U25.2, U26.2, U27.2, U28.2, U29.2, U30.2, U31.2, U32.2, U33.2, U34.2, U35.2, U36.2, U37.2, U38.2, U6.2, U7.2, U8.2, U9.2; no longer U1.1 (X4), U1.12 (X3), U1.13 (X0), U1.14 (X1), U1.15 (X2), U1.2 (X6), U1.4 (X7), U1.5 (X5), U2.1 (X4), U2.12 (X3), U2.13 (X0), U2.14 (X1), U2.15 (X2), U2.2 (X6), U2.4 (X7), U2.5 (X5), U3.1 (X4), U3.2 (X6), U3.4 (X7), U3.5 (X5), U4.1 (X4), U4.12 (X3), U4.13 (X0), U4.14 (X1), U4.15 (X2), U4.2 (X6), U4.4 (X7), U4.5 (X5), U5.12 (X3), U5.13 (X0), U5.14 (X1), U5.15 (X2), U5.5 (X5)
- new net X0: U1.5 (X5), U11.1
- new net X1: U1.4 (X7), U13.1
- new net X10: U2.4 (X7), U21.1
- new net X11: U19.1, U2.5 (X5)
- new net X12: U16.1, U2.15 (X2)
- new net X13: U15.1, U2.14 (X1)
- new net X14: U14.1, U2.13 (X0)
- new net X15: U17.1, U2.12 (X3)
- new net X16: U22.1, U3.1 (X4)
- new net X17: U24.1, U3.2 (X6)
- new net X18: U25.1, U3.4 (X7)
- new net X19: U23.1, U3.5 (X5)
- new net X2: U1.2 (X6), U12.1
- new net X3: U1.1 (X4), U10.1
- new net X4: U1.15 (X2), U8.1
- new net X5: U1.14 (X1), U7.1
- new net X6: U1.13 (X0), U6.1
- new net X7: U1.12 (X3), U9.1
- new net X8: U18.1, U2.1 (X4)
- new net X9: U2.2 (X6), U20.1
- new net Y0: U29.1, U4.12 (X3)
- new net Y1: U26.1, U4.13 (X0)
- new net Y10: U35.1, U5.14 (X1)
- new net Y11: U36.1, U5.15 (X2)
- new net Y12: U38.1, U5.5 (X5)
- new net Y2: U27.1, U4.14 (X1)
- new net Y3: U28.1, U4.15 (X2)
- new net Y4: U30.1, U4.1 (X4)
- new net Y5: U32.1, U4.2 (X6)
- new net Y6: U33.1, U4.4 (X7)
- new net Y7: U31.1, U4.5 (X5)
- new net Y8: U37.1, U5.12 (X3)
- new net Y9: U34.1, U5.13 (X0)
