File: kicad/wacom/wacom.kicad_pcb (KiCad board)
At the start: 2 copper layers, 56.5 x 40.6 mm, 33 parts, among them IC1 AVR128DB48, J1 UART, J2 TP1, J3 PORTB, J4 UPDI, J5 PORTF, J6 PORTA, J7 POWER, J8 WAC, SW1 RTS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

Commit message: images and python
Other:
- board text added: "JLCJLCJLC"
Changed lines of the file:
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@@
   (gr_line (start 144.78 56.515) (end 144.78 55.88) (layer "Edge.Cuts") (width 0.1))
   (gr_line (start 88.265 96.52) (end 144.78 96.52) (layer "Edge.Cuts") (width 0.1))
+  (gr_text "JLCJLCJLC\n" (at 90.932 70.358 270) (layer "F.SilkS")
+    (effects (font (size 1.5 1.5) (thickness 0.3)))
+  )
   (segment (start 112.102362 81.768) (end 111.574362 82.296) (width 0.2) (layer "F.Cu") (net 1))
   (segment (start 113.618 81.768) (end 112.102362 81.768) (width 0.2) (layer "F.Cu") (net 1))

Commit message: update
Parts:
- removed SW1: RTS, button:button
- added R9: 1k, Resistor_SMD:R_0603_1608Metric_Pad0.98x0.95mm_HandSolder, F.Cu at (100.8, 65.8)
- added REF**: TestPoint_Pad_D1.5mm, TestPoint:TestPoint_Pad_D1.5mm, F.Cu at (102.1, 83.6)
- added REF**: TestPoint_Pad_D1.5mm, TestPoint:TestPoint_Pad_D1.5mm, F.Cu at (109.7, 74.2)
- added REF**: TestPoint_Pad_D1.5mm, TestPoint:TestPoint_Pad_D1.5mm, F.Cu at (102.1, 86.2)
- J8: footprint Connector_PinHeader_2.54mm:PinHeader_2x09_P2.54mm_Vertical -> Connector_PinSocket_2.54mm:PinSocket_2x09_P2.54mm_Vertical
- R2: value 150 -> 10k
- R3: value 100 -> 820
- R4, R5: value 1k2 -> 10k
- R8: value 1k -> 10k
- moved R6 33.5 mm to (125.8, 85.7), turned to -90 degrees
- moved R8 14.8 mm to (105.7, 79.8), turned to 180 degrees
- moved J1 12.7 mm to (94.6, 65.4), turned to 0 degrees
- moved R3 10.8 mm to (112.8, 73.7), turned to 180 degrees
- moved R1 8.24 mm to (108.8, 83.3), turned to 0 degrees
- moved C1 7.79 mm to (102.6, 80.7), turned to 90 degrees
- moved R2 7.19 mm to (114.0, 71.9)
- moved R4 6.20 mm to (109.8, 81.8), turned to 0 degrees
- moved D1 5.09 mm to (105.4, 84.6), turned to -90 degrees
- moved R5 4.73 mm to (111.5, 77.2), turned to 90 degrees
- moved R7 4.07 mm to (109.5, 77.2), turned to -90 degrees
- moved D2 3.26 mm to (105.7, 81.5), turned to 0 degrees
- moved J8 2.54 mm to (142.2, 61.6)
- moved C7 0.51 mm to (110.2, 79.8)
- moved C8 0.13 mm to (116.3, 64.5)
Connections:
- C1 pad 1: /OP2- -> /OUT
- C1 pad 2: /OP2_OUT -> GND
- D1 pad 1: /OP2+ -> Net-(D1-Pad1)
- D1 pad 2: /OP1_OUT -> VCC
- D2 pad 1: /OP1_OUT -> /OUT
- D2 pad 2: Net-(D2-Pad2) -> /OP2_OUT
- IC1 pad 20: /OP2_OUT -> /OUT
- IC1 pad 24: /OP1+ -> /OUT
- R1 pad 1: GND -> Net-(D1-Pad1)
- R1 pad 2: /OP0_OUT -> /OP2-
- R2 pad 1: /OP0_OUT -> GND
- R2 pad 2: /OP1- -> /OP0_OUT
- R3 pad 1: /OP2- -> /OP0_OUT
- R3 pad 2: Net-(D2-Pad2) -> /OP1-
- R4 pad 1: /OP1- -> /OP2-
- R4 pad 2: /OP2+ -> /OP2_OUT
- R5 pad 2: Net-(D2-Pad2) -> /OP1_OUT
- R7 pad 1: GND -> /OP1_OUT
- R7 pad 2: /OP1_OUT -> /OP2+
- R8 pad 1: VCC -> /OP2+
- R8 pad 2: Net-(D3-Pad2) -> GND
Routing:
- net /RTS: track 79.6 -> 12.9 mm, vias 1 -> 2
- net /OUT: track 0.00 -> 34.7 mm, vias 0 -> 3
- net GND: track 80.5 -> 106.7 mm
- net /OP1_OUT: track 21.4 -> 6.90 mm
- net /S2: track 29.4 -> 19.0 mm
- net Net-(IC1-Pad5): track 30.9 -> 39.2 mm
- net Net-(D2-Pad2): track 6.58 -> 0.00 mm
- net /S0: track 24.0 -> 30.3 mm
- net /OP0_OUT: track 12.6 -> 7.18 mm
- net /ANALOG_B: track 34.3 -> 38.9 mm
- net /OP1-: track 9.43 -> 13.5 mm
- net /OP2_OUT: track 19.1 -> 15.3 mm, vias 2 -> 0
- net /CS1: track 32.5 -> 29.0 mm
- net /CS3: track 36.8 -> 33.2 mm
- net /CS0: track 19.5 -> 22.4 mm
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- removed copper zone on F.Cu, net GND
