File: kicad/wacom/wacom.kicad_sch (KiCad schematic)
At the start: 21 parts, among them IC1 AVR128DB48-I_PT, J1 UART, J2 TP1, J3 WAC, J4 POWER, U1 POWER_GEN

Commit message: python view
Connections:
- net GND: now also J3.1 (Pin_1), J3.2 (Pin_2)
- net VSS: now also J3.9 (Pin_9)
Changed lines of the file:
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@@
   (junction (at 59.69 133.35) (diameter 0) (color 0 0 0 0)
+  )
+  (junction (at 176.53 43.18) (diameter 0) (color 0 0 0 0)
   )
   (junction (at 111.76 69.85) (diameter 0) (color 0 0 0 0)
@@
     (stroke (width 0) (type default) (color 0 0 0 0))
   )
+  (wire (pts (xy 158.75 43.18) (xy 176.53 43.18))
+    (stroke (width 0) (type default) (color 0 0 0 0))
+  )
   (wire (pts (xy 102.87 69.85) (xy 111.76 69.85))
     (stroke (width 0) (type default) (color 0 0 0 0))
@@
   )
   (wire (pts (xy 80.01 73.025) (xy 88.9 73.025))
+    (stroke (width 0) (type default) (color 0 0 0 0))
+  )
+  (wire (pts (xy 164.465 60.96) (xy 176.53 60.96))
     (stroke (width 0) (type default) (color 0 0 0 0))
   )
@@
     (pin "2")
   )
+  (symbol (lib_id "power:GND") (at 158.75 43.18 0) (unit 1)
+    (in_bom yes) (on_board yes) (fields_autoplaced)
+    (property "Reference" "#PWR?" (id 0) (at 158.75 49.53 0)
+      (effects (font (size 1.27 1.27)) hide)
+    )
+    (property "Value" "GND" (id 1) (at 158.75 48.26 0))
+    (property "Footprint" "" (id 2) (at 158.75 43.18 0)
+      (effects (font (size 1.27 1.27)) hide)
+    )
+    (property "Datasheet" "" (id 3) (at 158.75 43.18 0)
+      (effects (font (size 1.27 1.27)) hide)
+    )
+    (pin "1")
+  )
   (symbol (lib_id "power:GND") (at 135.89 64.77 0) (unit 1)
     (in_bom yes) (on_board yes) (fields_autoplaced)
@@
     (pin "1")
     (pin "2")
+  )
+  (symbol (lib_id "power:VSS") (at 164.465 60.96 180) (unit 1)
+    (in_bom yes) (on_board yes) (fields_autoplaced)
+    (property "Reference" "#PWR?" (id 0) (at 164.465 57.15 0)
+      (effects (font (size 1.27 1.27)) hide)
+    )
+    (property "Value" "VSS" (id 1) (at 164.465 65.405 0))
+    (property "Footprint" "" (id 2) (at 164.465 60.96 0)
+      (effects (font (size 1.27 1.27)) hide)
+    )
+    (property "Datasheet" "" (id 3) (at 164.465 60.96 0)
+      (effects (font (size 1.27 1.27)) hide)
+    )
+    (pin "1")
   )
   (symbol (lib_id "Device:Opamp_Dual") (at 121.92 81.28 0) (unit 2)
@@
       (reference "#PWR017") (unit 1) (value "VSS") (footprint "")
     )
+    (path "/46648d41-7272-4121-8e6b-ccb621bdaefc"
+      (reference "#PWR?") (unit 1) (value "GND") (footprint "")
+    )
+    (path "/6a77db1c-7792-490c-b647-df6cd70d2a86"
+      (reference "#PWR?") (unit 1) (value "VSS") (footprint "")
+    )
     (path "/0c536bbb-c9a1-4003-8a25-0c190b4aea6b"

Commit message: pcb
Parts:
- removed J1: UART, Connector_PinHeader_2.54mm:PinHeader_1x03_P2.54mm_Vertical, symbol Connector:Conn_01x03_Male
- removed J3: WAC, Connector_PinHeader_2.54mm:PinHeader_1x18_P2.54mm_Vertical, symbol Connector:Conn_01x18_Female
- added C2, C3, C4: 100n, Capacitor_SMD:C_0603_1608Metric_Pad1.08x0.95mm_HandSolder, symbol Device:C
- added D3: LED, LED_SMD:LED_0603_1608Metric_Pad1.05x0.95mm_HandSolder, symbol Device:LED
- added J1: UART, Connector_PinHeader_2.54mm:PinHeader_1x06_P2.54mm_Vertical, symbol Connector:Conn_01x06_Male
- added J3: PORTB, Connector_PinHeader_2.54mm:PinHeader_1x04_P2.54mm_Vertical, symbol Connector:Conn_01x04_Male
- added J4: UPDI, Connector_PinHeader_2.54mm:PinHeader_2x03_P2.54mm_Vertical, symbol Connector_Generic:Conn_02x03_Odd_Even
- added J5: PORTF, Connector_PinHeader_2.54mm:PinHeader_1x04_P2.54mm_Vertical, symbol Connector:Conn_01x04_Male
- added J6: PORTA, Connector_PinHeader_2.54mm:PinHeader_1x08_P2.54mm_Vertical, symbol Connector:Conn_01x08_Male
- added J8: WAC, Connector_PinHeader_2.54mm:PinHeader_2x09_P2.54mm_Vertical, symbol Connector:Conn_01x18_Female
- added JP1: PF0_ANA, Jumper:SolderJumper-2_P1.3mm_Open_RoundedPad1.0x1.5mm, symbol Jumper:SolderJumper_2_Open
- added R6: 10k, Resistor_SMD:R_0603_1608Metric_Pad0.98x0.95mm_HandSolder, symbol Device:R
- added R8: 1k, Resistor_SMD:R_0603_1608Metric_Pad0.98x0.95mm_HandSolder, symbol Device:R
- added SW1: RTS, button:button, symbol Switch:SW_Push
- C1: value 100n -> 1u
- C10: renamed from C7; footprint (none) -> Capacitor_SMD:C_0603_1608Metric_Pad1.08x0.95mm_HandSolder
- C8: renamed from C5; footprint (none) -> Capacitor_SMD:C_0603_1608Metric_Pad1.08x0.95mm_HandSolder
- C9: renamed from C6; value 10u -> 100n; footprint (none) -> Capacitor_SMD:C_0603_1608Metric_Pad1.08x0.95mm_HandSolder
- D1, D2: footprint (none) -> Diode_SMD:D_SOD-323_HandSoldering
- IC1: value AVR128DB48-I_PT -> AVR128DB48; footprint QFP50P900X900X120-48N -> AVR128DB48-I_PT:QFP50P900X900X120-48N
- R2: value 330 -> 150
- renumbered C2 to C5, C3 to C6, C4 to C7, J4 to J7, R6 to R7
Connections:
- net ANALOG_A: now also J8.4 (Pin_4), J8.5 (Pin_5), JP1.2 (B)
- net ANALOG_B: now also J8.3 (Pin_3)
- net CS0: now also J8.13 (Pin_13)
- net CS1: now also J8.14 (Pin_14)
- net CS2: now also J8.15 (Pin_15)
- net CS3: now also J8.16 (Pin_16)
- net CS4: now also J8.17 (Pin_17)
- net GND: now also J8.1 (Pin_1), J8.2 (Pin_2)
- net S0: now also J8.10 (Pin_10)
- net S1: now also J8.11 (Pin_11)
- net S2: now also J8.12 (Pin_12)
- net VCC: now also IC1.14 (VDDIO2), IC1.28 (AVDD), IC1.42 (VDD), C2.1, C3.1, C4.1, J1.4 (Pin_4), J4.2 (Pin_2), J8.7 (Pin_7), J8.8 (Pin_8), R6.1, R8.1
- net VSS: now also IC1.15 (GND_1), IC1.29 (GND_2), IC1.43 (GND_3), C2.2, C3.2, C4.2, D3.1 (K), J1.1 (Pin_1), J1.6 (Pin_6), J4.6 (Pin_6), J8.9 (Pin_9), SW1.2
- net PA5: now reaches IC1.1 (PA5)
- net PA5: now also J6.6 (Pin_6)
- net PA6: now reaches IC1.2 (PA6)
- net PA6: now also J6.7 (Pin_7)
- net PA7: now reaches IC1.3 (PA7)
- net PA7: now also J6.8 (Pin_8)
- net PF0: now reaches IC1.34 (PF0(XTAL32K1))
- net PF0: now also J5.1 (Pin_1), JP1.1 (A)
- net PF1: now reaches IC1.35 (PF1(XTAL32K2))
- net PF1: now also J5.2 (Pin_2)
- net PF2: now reaches IC1.36 (PF2)
- net PF2: now also J5.3 (Pin_3)
- net PF3: now reaches IC1.37 (PF3)
- net PF3: now also J5.4 (Pin_4)
- net at IC1.4 (PB0): now also J1.2 (Pin_2)
- net RTS: now reaches IC1.40 (PF6)
- net RTS: now also R6.2, SW1.1
- net UPDI: now reaches IC1.41 (UPDI)
- net UPDI: now also J4.1 (Pin_1)
- net PA0: now reaches IC1.44 (PA0(XTALHF1))
- net PA0: now also J6.1 (Pin_1)
- net PA1: now reaches IC1.45 (PA1(XTALHF2))
- net PA1: now also J6.2 (Pin_2)
- net PA2: now reaches IC1.46 (PA2)
- net PA2: now also J6.3 (Pin_3)
- net PA3: now reaches IC1.47 (PA3)
- net PA3: now also J6.4 (Pin_4)
- net PA4: now reaches IC1.48 (PA4)
- net PA4: now also J6.5 (Pin_5)
- net at IC1.5 (PB1): now also J1.3 (Pin_3)
- net PB2: now reaches IC1.6 (PB2)
- net PB2: now also J3.1 (Pin_1)
- net PB3: now reaches IC1.7 (PB3)
- net PB3: now also J3.2 (Pin_2)
- net PB4: now reaches IC1.8 (PB4)
- net PB4: now also J3.3 (Pin_3)
- net PB5: now reaches IC1.9 (PB5)
- net PB5: now also J3.4 (Pin_4)
- new net: D3.2 (A), R8.2
- no-connect marks 2 -> 6
Other:
- note added: "Near MCU"
- moved on the sheet: C1, D1, D2, R1, R2, R3, R4, R5, R7

Commit message: update
Parts:
- removed R5: 1k2, Resistor_SMD:R_0603_1608Metric_Pad0.98x0.95mm_HandSolder, symbol Device:R
- removed SW1: RTS, button:button, symbol Switch:SW_Push
- added R1, R8: 10k, Resistor_SMD:R_0603_1608Metric_Pad0.98x0.95mm_HandSolder, symbol Device:R
- J8: footprint Connector_PinHeader_2.54mm:PinHeader_2x09_P2.54mm_Vertical -> Connector_PinSocket_2.54mm:PinSocket_2x09_P2.54mm_Vertical
- R3: renamed from R2; value 150 -> 820
- R4: renamed from R3; value 100 -> 10k
- R5: renamed from R4; value 1k2 -> 10k
- renumbered R1 to R2, R8 to R9
Connections:
- net GND: now also C1.2, R8.2; no longer R7.1
- net OP1_OUT: now also R5.2, R7.1; no longer D1.2 (A), D2.1 (K), R7.2
- net OP2+: now also R7.2, R8.1; no longer D1.1 (K), R5.2
- net OP2-: now also R1.2; no longer C1.1
- net OP2_OUT: now also D2.2 (A), R4.2; no longer C1.2, IC1.20 (PD0)
- net VCC: now also D1.2 (A)
- net OP1+ renamed OUT
- net OUT: now also C1.1, D2.1 (K), IC1.20 (PD0)
- new net: D1.1 (K), R1.1
Other:
- moved on the sheet: C1, D2
